File: golden/golden_led_button.kicad_sch (KiCad schematic)
At the start: 3 parts, among them SW1 SW_Push

Commit message: Step 2: footprint index + pin/pad validation + deterministic auto-assignment
Official kicad-footprints clone (15,448 .kicad_mod) indexed into
parts.sqlite: descr/tags/attr, distinct pad numbers per footprint
(fp_pads). New fp_checks module:
- check_footprints: footprint must exist AND every symbol pin NUMBER must
  have a pad (number matching, not count) — completes the §8.2
  'footprint pin mismatch' rule that free-text footprints made impossible
- assign_footprints: empty/invalid footprints filled deterministically —
  symbol default Footprint property first, then ki_fp_filters glob match
  (0805 > 0603 preference for common passives)

Wired into pipeline (parts_index param) and agent (after synthesis and
every repair round). First live catch was our own fixture: golden's
'SW_SPST_PTS645' never existed — real name SW_SPST_PTS645Sx43SMTR92,
fixed everywhere and golden regenerated. Live run: model footprints
auto-corrected to LED_SMD/Resistor_SMD 0805, ERC 0. 68 tests green.

Co-Authored-By: Claude Fable 5 <noreply@anthropic.com>
Parts:
- SW1: footprint Button_Switch_SMD:SW_SPST_PTS645 -> Button_Switch_SMD:SW_SPST_PTS645Sx43SMTR92
Changed lines of the file:
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@@
 			)
 		)
-		(property "Footprint" "Button_Switch_SMD:SW_SPST_PTS645"
+		(property "Footprint" "Button_Switch_SMD:SW_SPST_PTS645Sx43SMTR92"
 			(at 63.5 63.5 0)
 			(show_name no)
